File: traffic_light.brd (EAGLE design)
At the start: 19 x 47.2 mm, 18 parts

Commit message: Update readme and all the things
Changed lines of the file:
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@@
 <?xml version="1.0" encoding="utf-8"?>
 <!DOCTYPE eagle SYSTEM "eagle.dtd">
-<eagle version="9.1.0">
+<eagle version="9.4.0">
 <drawing>
 <settings>
@@
 <layer number="56" name="wert" color="7" fill="1" visible="no" active="no"/>
 <layer number="57" name="tCAD" color="7" fill="1" visible="no" active="no"/>
+<layer number="58" name="tCAD" color="7" fill="1" visible="no" active="no"/>
 <layer number="59" name="tCarbon" color="7" fill="1" visible="no" active="no"/>
 <layer number="60" name="bCarbon" color="7" fill="1" visible="no" active="no"/>
@@
 <layer number="131" name="tAdjust" color="7" fill="1" visible="yes" active="yes"/>
 <layer number="132" name="bAdjust" color="7" fill="1" visible="yes" active="yes"/>
+<layer number="133" name="bottom_silk" color="7" fill="1" visible="yes" active="yes"/>
 <layer number="144" name="Drill_legend" color="7" fill="1" visible="yes" active="yes"/>
+<layer number="145" name="DrillLegend_01-16" color="2" fill="9" visible="no" active="yes"/>
 <layer number="150" name="Notes" color="7" fill="1" visible="yes" active="yes"/>
 <layer number="151" name="HeatSink" color="7" fill="1" visible="yes" active="yes"/>
@@
 <wire x1="18.5" y1="35" x2="-0.5" y2="35" width="0" layer="20"/>
 <wire x1="-0.5" y1="35" x2="-0.5" y2="0" width="0" layer="20"/>
-<hole x="9" y="25" drill="2"/>
 <hole x="3" y="7" drill="2"/>
 <hole x="4" y="2" drill="1.5"/>
@@
 </autorouter>
 <elements>
-<element name="D1" library="SparkFun-LED" package="LED-0603" value="RED" x="9" y="30" rot="MR270"/>
-<element name="D2" library="SparkFun-LED" package="LED-0603" value="AMBER" x="9" y="17.5" rot="MR270"/>
-<element name="D3" library="SparkFun-LED" package="LED-0603" value="GREEN" x="9" y="5" rot="MR270"/>
-<element name="MDL1" library="ESP8266-ESP12E" package="ESP8266-ESP12E" value="" x="0.889" y="10.414"/>
-<element name="C1" library="rcl" package="C0805" value="0.1uf" x="4.572" y="12.954" rot="MR180"/>
-<element name="R1" library="rcl" package="R0805" value="150" x="4.572" y="22.606" rot="MR180"/>
-<element name="R4" library="rcl" package="R0805" value="10k" x="4.572" y="31.75" rot="MR0"/>
-<element name="R5" library="rcl" package="R0805" value="10k" x="4.572" y="24.892" rot="MR0"/>
-<element name="R6" library="rcl" package="R0805" value="10k" x="13.97" y="18.288" rot="MR180"/>
-<element name="R7" library="rcl" package="R0805" value="10k" x="13.97" y="16.002" rot="MR180"/>
-<element name="LOGO1" library="SparkFun-Aesthetics" package="OSHW-LOGO-S" value="OSHW-LOGOS" x="16.002" y="5.334"/>
-<element name="J2" library="SparkFun-Connectors" package="2X3-SHROUDED" value="" x="8.636" y="-7.62" rot="R90">
+<element name="D1" library="SparkFun-LED" package="LED-0603" value="RED" x="9" y="30" smashed="yes" rot="MR270">
+<attribute name="NAME" x="9.889" y="30.6985" size="0.4064" layer="26" rot="MR0"/>
+<attribute name="VALUE" x="10.016" y="28.9205" size="0.4064" layer="28" rot="MR0"/>
+</element>
+<element name="D2" library="SparkFun-LED" package="LED-0603" value="AMBER" x="9" y="17.5" smashed="yes" rot="MR270">
+<attribute name="NAME" x="9.889" y="18.1985" size="0.4064" layer="26" rot="MR0"/>
+<attribute name="VALUE" x="10.016" y="16.4205" size="0.4064" layer="28" rot="MR0"/>
+</element>
+<element name="D3" library="SparkFun-LED" package="LED-0603" value="GREEN" x="9" y="5" smashed="yes" rot="MR270">
+<attribute name="NAME" x="9.889" y="5.6985" size="0.4064" layer="26" rot="MR0"/>
+<attribute name="VALUE" x="10.016" y="3.9205" size="0.4064" layer="28" rot="MR0"/>
+</element>
+<element name="MDL1" library="ESP8266-ESP12E" package="ESP8266-ESP12E" value="" x="0.889" y="10.414" smashed="yes">
+<attribute name="NAME" x="5.889" y="12.414" size="1.27" layer="21" rot="R90"/>
+</element>
+<element name="C1" library="rcl" package="C0805" value="0.1uf" x="4.572" y="12.954" smashed="yes" rot="MR180">
+<attribute name="NAME" x="3.302" y="11.684" size="1.27" layer="26" rot="MR180"/>
+<attribute name="VALUE" x="3.302" y="15.494" size="1.27" layer="28" rot="MR180"/>
+</element>
+<element name="R1" library="rcl" package="R0805" value="150" x="4.572" y="22.606" smashed="yes" rot="MR180">
+<attribute name="NAME" x="3.937" y="21.336" size="1.27" layer="26" rot="MR180"/>
+<attribute name="VALUE" x="3.937" y="25.146" size="1.27" layer="28" rot="MR180"/>
+</element>
+<element name="R4" library="rcl" package="R0805" value="10k" x="4.572" y="31.75" smashed="yes" rot="MR0">
+<attribute name="NAME" x="5.207" y="33.02" size="1.27" layer="26" rot="MR0"/>
+<attribute name="VALUE" x="5.207" y="29.21" size="1.27" layer="28" rot="MR0"/>
+</element>
+<element name="R5" library="rcl" package="R0805" value="10k" x="4.572" y="24.892" smashed="yes" rot="MR0">
+<attribute name="NAME" x="5.207" y="26.162" size="1.27" layer="26" rot="MR0"/>
+<attribute name="VALUE" x="5.207" y="22.352" size="1.27" layer="28" rot="MR0"/>
+</element>
+<element name="R6" library="rcl" package="R0805" value="10k" x="13.97" y="18.288" smashed="yes" rot="MR180">
+<attribute name="NAME" x="13.335" y="17.018" size="1.27" layer="26" rot="MR180"/>
+<attribute name="VALUE" x="13.335" y="20.828" size="1.27" layer="28" rot="MR180"/>
+</element>
+<element name="R7" library="rcl" package="R0805" value="10k" x="13.97" y="16.002" smashed="yes" rot="MR180">
+<attribute name="NAME" x="13.335" y="14.732" size="1.27" layer="26" rot="MR180"/>
+<attribute name="VALUE" x="13.335" y="18.542" size="1.27" layer="28" rot="MR180"/>
+</element>
+<element name="LOGO1" library="SparkFun-Aesthetics" package="OSHW-LOGO-S" value="OSHW-LOGOS" x="16.002" y="5.334" smashed="yes"/>
+<element name="J2" library="SparkFun-Connectors" package="2X3-SHROUDED" value="" x="8.636" y="-7.62" smashed="yes" rot="R90">
+<attribute name="NAME" x="0.762" y="-11.43" size="0.6096" layer="25" font="vector" ratio="20" rot="R90"/>
 <attribute name="PROD_ID" value="CONN-10681" x="-15.24" y="-29.21" size="0.6096" layer="27" rot="R90" display="off"/>
 <attribute name="SF_ID" value="PRT_10877" x="-15.24" y="-29.21" size="0.6096" layer="27" rot="R90" display="off"/>
-</element>
-<element name="R2" library="rcl" package="R0805" value="150" x="4.572" y="20.32" rot="MR180"/>
-<element name="R3" library="rcl" package="R0805" value="120" x="4.572" y="18.034" rot="MR180"/>
-<element name="R8" library="rcl" package="R0805" value="390k" x="4.572" y="27.178" rot="MR180"/>
-<element name="R9" library="rcl" package="R0805" value="100k" x="4.572" y="29.464" rot="MR0"/>
+<attribute name="VALUE" x="17.018" y="-11.43" size="0.6096" layer="27" font="vector" ratio="20" rot="R90"/>
+</element>
+<element name="R2" library="rcl" package="R0805" value="150" x="4.572" y="20.32" smashed="yes" rot="MR180">
+<attribute name="NAME" x="3.937" y="19.05" size="1.27" layer="26" rot="MR180"/>
+<attribute name="VALUE" x="3.937" y="22.86" size="1.27" layer="28" rot="MR180"/>
+</element>
+<element name="R3" library="rcl" package="R0805" value="120" x="4.572" y="18.034" smashed="yes" rot="MR180">
+<attribute name="NAME" x="3.937" y="16.764" size="1.27" layer="26" rot="MR180"/>
+<attribute name="VALUE" x="3.937" y="20.574" size="1.27" layer="28" rot="MR180"/>
+</element>
+<element name="R8" library="rcl" package="R0805" value="390k" x="4.572" y="27.178" smashed="yes" rot="MR180">
+<attribute name="NAME" x="3.937" y="25.908" size="1.27" layer="26" rot="MR180"/>
+<attribute name="VALUE" x="3.937" y="29.718" size="1.27" layer="28" rot="MR180"/>
+</element>
+<element name="R9" library="rcl" package="R0805" value="100k" x="4.572" y="29.464" smashed="yes" rot="MR0">
+<attribute name="NAME" x="5.207" y="30.734" size="1.27" layer="26" rot="MR0"/>
+<attribute name="VALUE" x="5.207" y="26.924" size="1.27" layer="28" rot="MR0"/>
+</element>
 <element name="V_BATT" library="wirepad" library_urn="urn:adsk.eagle:library:412" package="SMD2,54-5,08" package3d_urn="urn:adsk.eagle:package:30841/1" value="" x="2.794" y="2.032" smashed="yes" rot="R270">
 <attribute name="NAME" x="0.294" y="3.532" size="0.8128" layer="25"/>
@@
 <wire x1="7.874" y1="7.71104375" x2="7.874" y2="10.602" width="0.254" layer="16"/>
 <polygon width="0.254" layer="1">
-<vertex x="-1.016" y="37.846"/>
-<vertex x="22.606" y="37.846"/>
-<vertex x="23.114" y="0"/>
+<vertex x="-2.032" y="38.1"/>
+<vertex x="20.574" y="38.1"/>
+<vertex x="20.574" y="0"/>
 <vertex x="-2.032" y="0"/>
 </polygon>
@@
 <via x="12.446" y="8.128" extent="1-16" drill="0.35"/>
 <polygon width="0.254" layer="16">
-<vertex x="-2.794" y="39.878"/>
-<vertex x="19.05" y="39.878"/>
-<vertex x="19.05" y="0"/>
-<vertex x="-2.794" y="0"/>
+<vertex x="-2.667" y="38.735"/>
+<vertex x="21.209" y="38.735"/>
+<vertex x="21.209" y="0"/>
+<vertex x="-2.667" y="0"/>
 </polygon>
 </signal>
