File: traffic_light.sch (EAGLE design)
At the start: 18 parts

Commit message: Update readme and all the things
Other:
- note removed: "Processor"
- note removed: "Pullups"
- moved on the sheet: C1, D1, D2, D3, GND, J2, MDL1, R1, R2, R3, R4, R5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
