File: usb_power.sch (EAGLE design)
At the start: 6 parts, among them U1 REG1117-3.3

Commit message: Update readme and all the things
Changed lines of the file:
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@@
 <?xml version="1.0" encoding="utf-8"?>
 <!DOCTYPE eagle SYSTEM "eagle.dtd">
-<eagle version="9.0.1">
+<eagle version="9.4.0">
 <drawing>
 <settings>
@@
 <layer number="56" name="wert" color="7" fill="1" visible="no" active="no"/>
 <layer number="57" name="tCAD" color="7" fill="1" visible="no" active="no"/>
+<layer number="58" name="tCAD" color="7" fill="1" visible="no" active="no"/>
 <layer number="59" name="tCarbon" color="7" fill="1" visible="no" active="no"/>
 <layer number="60" name="bCarbon" color="7" fill="1" visible="no" active="no"/>
@@
 <layer number="115" name="ReferenceISLANDS" color="7" fill="1" visible="yes" active="yes"/>
 <layer number="116" name="Patch_BOT" color="9" fill="4" visible="yes" active="yes"/>
+<layer number="117" name="BACKMAAT1" color="7" fill="1" visible="yes" active="yes"/>
 <layer number="118" name="Rect_Pads" color="7" fill="1" visible="yes" active="yes"/>
+<layer number="119" name="KAP_TEKEN" color="7" fill="1" visible="yes" active="yes"/>
+<layer number="120" name="120" color="7" fill="1" visible="yes" active="yes"/>
 <layer number="121" name="_tsilk" color="7" fill="1" visible="yes" active="yes"/>
 <layer number="122" name="_bsilk" color="7" fill="1" visible="yes" active="yes"/>
@@
 <layer number="128" name="_bValues" color="7" fill="1" visible="yes" active="yes"/>
 <layer number="129" name="Mask" color="7" fill="1" visible="yes" active="yes"/>
+<layer number="130" name="SMDSTROOK" color="7" fill="1" visible="yes" active="yes"/>
 <layer number="131" name="tAdjust" color="7" fill="1" visible="yes" active="yes"/>
 <layer number="132" name="bAdjust" color="7" fill="1" visible="yes" active="yes"/>
+<layer number="133" name="bottom_silk" color="7" fill="1" visible="yes" active="yes"/>
 <layer number="144" name="Drill_legend" color="7" fill="1" visible="yes" active="yes"/>
+<layer number="145" name="DrillLegend_01-16" color="2" fill="9" visible="no" active="yes"/>
 <layer number="150" name="Notes" color="7" fill="1" visible="yes" active="yes"/>
 <layer number="151" name="HeatSink" color="7" fill="1" visible="yes" active="yes"/>
@@
 <part name="PAD1" library="wirepad" library_urn="urn:adsk.eagle:library:412" deviceset="SMD5" device="" package3d_urn="urn:adsk.eagle:package:30841/1"/>
 <part name="PAD2" library="wirepad" library_urn="urn:adsk.eagle:library:412" deviceset="SMD5" device="" package3d_urn="urn:adsk.eagle:package:30841/1"/>
+<part name="FRAME1" library="SparkFun-Aesthetics" library_urn="urn:adsk.eagle:library:507" deviceset="FRAME-A4L" device=""/>
 </parts>
 <sheets>
@@
 </plain>
 <instances>
-<instance part="J1" gate="G$1" x="-10.16" y="30.48" rot="MR0"/>
-<instance part="SUPPLY1" gate="G$1" x="55.88" y="43.18"/>
-<instance part="U1" gate="A" x="30.48" y="30.48"/>
-<instance part="GND1" gate="1" x="2.54" y="12.7"/>
-<instance part="C1" gate="G$1" x="55.88" y="22.86"/>
-<instance part="C2" gate="G$1" x="2.54" y="33.02"/>
-<instance part="GND2" gate="1" x="55.88" y="7.62"/>
-<instance part="PAD1" gate="1" x="73.66" y="30.48" rot="R180"/>
-<instance part="PAD2" gate="1" x="73.66" y="15.24" rot="R180"/>
+<instance part="J1" gate="G$1" x="-10.16" y="30.48" smashed="yes" rot="MR0">
+<attribute name="VALUE" x="-7.62" y="22.606" size="1.778" layer="96" font="vector" rot="MR0" align="top-left"/>
+<attribute name="NAME" x="-7.62" y="38.1" size="1.778" layer="95" font="vector" rot="MR0"/>
+</instance>
+<instance part="SUPPLY1" gate="G$1" x="55.88" y="43.18" smashed="yes">
+<attribute name="VALUE" x="55.88" y="45.974" size="1.778" layer="96" align="bottom-center"/>
+</instance>
+<instance part="U1" gate="A" x="30.48" y="30.48" smashed="yes">
+<attribute name="NAME" x="25.1206" y="39.5986" size="2.0828" layer="95" ratio="10" rot="SR0"/>
+<attribute name="VALUE" x="26.9494" y="16.4846" size="2.0828" layer="96" ratio="10" rot="SR0"/>
+</instance>
+<instance part="GND1" gate="1" x="2.54" y="12.7" smashed="yes">
+<attribute name="VALUE" x="2.54" y="12.446" size="1.778" layer="96" align="top-center"/>
+</instance>
+<instance part="C1" gate="G$1" x="55.88" y="22.86" smashed="yes">
+<attribute name="NAME" x="56.896" y="23.495" size="1.778" layer="95" font="vector"/>
+<attribute name="VALUE" x="56.896" y="18.669" size="1.778" layer="96" font="vector"/>
+</instance>
+<instance part="C2" gate="G$1" x="2.54" y="33.02" smashed="yes">
+<attribute name="NAME" x="3.556" y="33.655" size="1.778" layer="95" font="vector"/>
+<attribute name="VALUE" x="3.556" y="28.829" size="1.778" layer="96" font="vector"/>
+</instance>
+<instance part="GND2" gate="1" x="55.88" y="7.62" smashed="yes">
+<attribute name="VALUE" x="55.88" y="7.366" size="1.778" layer="96" align="top-center"/>
+</instance>
+<instance part="PAD1" gate="1" x="73.66" y="30.48" smashed="yes" rot="R180">
+<attribute name="NAME" x="74.803" y="28.6258" size="1.778" layer="95" rot="R180"/>
+<attribute name="VALUE" x="74.803" y="33.782" size="1.778" layer="96" rot="R180"/>
+</instance>
+<instance part="PAD2" gate="1" x="73.66" y="15.24" smashed="yes" rot="R180">
+<attribute name="NAME" x="74.803" y="13.3858" size="1.778" layer="95" rot="R180"/>
+<attribute name="VALUE" x="74.803" y="18.542" size="1.778" layer="96" rot="R180"/>
+</instance>
+<instance part="FRAME1" gate="G$1" x="-101.6" y="-66.04" smashed="yes">
+<attribute name="DRAWING_NAME" x="80.01" y="-54.61" size="2.54" layer="94" font="vector"/>
+<attribute name="LAST_DATE_TIME" x="80.01" y="-59.69" size="2.286" layer="94" font="vector"/>
+<attribute name="SHEET" x="93.98" y="-64.77" size="2.54" layer="94" font="vector"/>
+</instance>
 </instances>
 <busses>
